Commit message: Adjustable camera angle to be done

File: src/simplecar.urdf (robot description, URDF)
Before this commit: robot simplecar, 7 links, 6 joints
Links:
- added link camera_link; collision cylinder length=0.07 radius=0.02; visual cylinder length=0.05 radius=0.02
- added link camera_mount_link; collision box size=0.1 0.1 0.1; visual box size=0.1 0.1 0.1
- added link camera_rod_link; collision box size=0.05 0.05 0.5; visual box size=0.05 0.05 0.5
Joints:
- added joint camera_joint: type revolute, parent camera_mount_link, child camera_link, origin xyz=0.05 0 0, axis 0 1 0, limit lower=0 upper=1
- added joint camera_mount_joint: type prismatic, parent camera_rod_link, child camera_mount_link, origin xyz=0 0 0, axis 0 0 1, limit lower=-0.1 upper=0.5
- added joint camera_rod_joint: type fixed, parent base_link, child camera_rod_link, origin xyz=0.1 0 0.3, axis 0 0 1

Commit message: redone the panel view but some bugs when client accpets commands

File: src/simplecar.urdf (robot description, URDF)
Before this commit: robot simplecar, 10 links, 9 joints
Joints:
- joint camera_mount_joint: limit lower=-0.1 upper=0.5 -> lower=0.1 upper=0.25

Commit message: many details

File: src/simplecar.urdf (robot description, URDF)
Before this commit: robot simplecar, 10 links, 9 joints
Links:
- link base_link: mass 6 -> 100

Commit message: changing sizes and uploaded a photo

File: src/simplecar.urdf (robot description, URDF)
Before this commit: robot simplecar, 10 links, 9 joints
Links:
- link base_link: mass 100 -> 6

Commit message: changed size of car

File: src/simplecar.urdf (robot description, URDF)
Before this commit: robot simplecar, 10 links, 9 joints
Links:
- link base_link: geometry collision box size=0.25 0.15 0.05; visual box size=0.25 0.15 0.05
- link camera_link: geometry collision cylinder length=0.025 radius=0.01; visual cylinder length=0.025 radius=0.01
- link camera_mount_link: geometry collision box size=0.05 0.05 0.05; visual box size=0.05 0.05 0.05
- link camera_rod_link: geometry collision box size=0.025 0.025 0.25; visual box size=0.025 0.025 0.25
- link left_back_wheel: geometry collision cylinder length=0.025 radius=0.05; visual cylinder length=0.025 radius=0.05
- link left_front_wheel: geometry collision cylinder length=0.025 radius=0.05; visual cylinder length=0.025 radius=0.05
- link left_hinge: geometry visual box size=0.1 0.01 0.01
- link right_back_wheel: geometry collision cylinder length=0.025 radius=0.05; visual cylinder length=0.025 radius=0.05
- link right_front_wheel: geometry collision cylinder length=0.025 radius=0.05; visual cylinder length=0.025 radius=0.05
- link right_hinge: geometry visual box size=0.1 0.01 0.01
Joints:
- joint base_to_left_back_wheel: origin xyz=-0.2 0.175 0 -> xyz=-0.1 0.0875 0
- joint base_to_left_hinge: origin xyz=0.2 0.0 0 -> xyz=0.1 0.0 0
- joint base_to_right_back_wheel: origin xyz=-0.2 -0.175 0 -> xyz=-0.1 -0.0875 0
- joint base_to_right_hinge: origin xyz=0.2 0 0 -> xyz=0.1 0 0
- joint camera_joint: origin xyz=0.05 0 0 -> xyz=0.025 0 0
- joint camera_rod_joint: origin xyz=0.1 0 0.3 -> xyz=0.05 0 0.15
- joint left_hinge_to_left_front_wheel: origin xyz=0 0.2 0 -> xyz=0 0.1 0
- joint right_hinge_to_right_front_wheel: origin xyz=0 -0.2 0 -> xyz=0 -0.1 0
